File: audio-rf/audio-rf.sch (KiCad schematic (older format))
At the start: 28 parts, among them J3 Conn_01x01, J4 Conn_01x01, J5 Conn_01x01, Q1 2N4401, SW2 SW_SPST, U3 LM386

Commit message: Associate footprints for all-through-hole
Parts:
- removed AE1: Antenna, symbol Device:Antenna
- added J6: Conn_Coaxial, homebrew:MOLEX_0731713150, symbol Connector:Conn_Coaxial
- C10, C8: value 1nF -> 1000pF; footprint (none) -> Capacitor_THT:C_Disc_D5.0mm_W2.5mm_P5.00mm
- C11: value 100nF -> 0.1uF; footprint (none) -> Capacitor_THT:C_Disc_D5.1mm_W3.2mm_P5.00mm
- C12: value 4.7nF -> 4700pF; footprint (none) -> Capacitor_THT:C_Disc_D5.1mm_W3.2mm_P5.00mm
- C13: value CP -> 10uF; footprint (none) -> Capacitor_THT:CP_Radial_D5.0mm_P2.00mm
- C14: value 47nF -> 47000pF; footprint (none) -> Capacitor_THT:C_Disc_D3.8mm_W2.6mm_P2.50mm
- C15: footprint (none) -> Capacitor_THT:CP_Radial_D6.3mm_P2.50mm
- C16, C9: footprint (none) -> Capacitor_THT:CP_Radial_D5.0mm_P2.00mm
- C7: footprint (none) -> Capacitor_THT:C_Disc_D5.0mm_W2.5mm_P5.00mm
- D3: footprint (none) -> Diode_THT:D_DO-35_SOD27_P7.62mm_Horizontal
- J3, J4, J5: footprint (none) -> Connector_PinHeader_2.54mm:PinHeader_1x01_P2.54mm_Vertical
- LS1: footprint (none) -> homebrew:CLS0231MP-1_SPEAKER
- R10, R11, R12, R13, R6, R7, R8, R9: footprint (none) -> Resistor_THT:R_Axial_DIN0207_L6.3mm_D2.5mm_P10.16mm_Horizontal
- RV1: footprint (none) -> Potentiometer_THT:Potentiometer_Bourns_PTV09A-2_Single_Horizontal
- SW2: footprint (none) -> homebrew:‎EG1206‎_SLIDE_SWITCH
- U3: footprint (none) -> Package_DIP:DIP-8_W7.62mm_Socket
Changed lines of the file:
@@
 F 0 "R12" V 4893 3150 50  0000 C CNN
 F 1 "1.2k" V 4984 3150 50  0000 C CNN
-F 2 "" V 5030 3150 50  0001 C CNN
+F 2 "Resistor_THT:R_Axial_DIN0207_L6.3mm_D2.5mm_P10.16mm_Horizontal" V 5030 3150 50  0001 C CNN
 F 3 "~" H 5100 3150 50  0001 C CNN
 	1    5100 3150
@@
 F 0 "SW2" H 4450 3385 50  0000 C CNN
 F 1 "SW_SPST" H 4450 3294 50  0000 C CNN
-F 2 "" H 4450 3150 50  0001 C CNN
+F 2 "homebrew:‎EG1206‎_SLIDE_SWITCH" H 4450 3150 50  0001 C CNN
 F 3 "~" H 4450 3150 50  0001 C CNN
 	1    4450 3150
@@
 P 4800 3150
 F 0 "C13" V 5055 3150 50  0000 C CNN
-F 1 "CP" V 4964 3150 50  0000 C CNN
-F 2 "" H 4838 3000 50  0001 C CNN
+F 1 "10uF" V 4964 3150 50  0000 C CNN
+F 2 "Capacitor_THT:CP_Radial_D5.0mm_P2.00mm" H 4838 3000 50  0001 C CNN
 F 3 "~" H 4800 3150 50  0001 C CNN
 	1    4800 3150
@@
 F 0 "LS1" H 6670 2196 50  0000 L CNN
 F 1 "Speaker" H 6670 2105 50  0000 L CNN
-F 2 "" H 6500 2000 50  0001 C CNN
+F 2 "homebrew:CLS0231MP-1_SPEAKER" H 6500 2000 50  0001 C CNN
 F 3 "~" H 6490 2150 50  0001 C CNN
 	1    6500 2200
@@
 F 0 "C15" V 6305 2200 50  0000 C CNN
 F 1 "220uF" V 6214 2200 50  0000 C CNN
-F 2 "" H 6088 2050 50  0001 C CNN
+F 2 "Capacitor_THT:CP_Radial_D6.3mm_P2.50mm" H 6088 2050 50  0001 C CNN
 F 3 "~" H 6050 2200 50  0001 C CNN
 	1    6050 2200
@@
 F 0 "C9" H 3068 1246 50  0000 L CNN
 F 1 "1uF" H 3068 1155 50  0000 L CNN
-F 2 "" H 2988 1050 50  0001 C CNN
+F 2 "Capacitor_THT:CP_Radial_D5.0mm_P2.00mm" H 2988 1050 50  0001 C CNN
 F 3 "~" H 2950 1200 50  0001 C CNN
 	1    2950 1200
@@
 P 5700 2700
 F 0 "C14" H 5815 2746 50  0000 L CNN
-F 1 "47nF" H 5815 2655 50  0000 L CNN
-F 2 "" H 5738 2550 50  0001 C CNN
+F 1 "47000pF" H 5815 2655 50  0000 L CNN
+F 2 "Capacitor_THT:C_Disc_D3.8mm_W2.6mm_P2.50mm" H 5738 2550 50  0001 C CNN
 F 3 "~" H 5700 2700 50  0001 C CNN
 	1    5700 2700
@@
 F 0 "R13" H 5770 2446 50  0000 L CNN
 F 1 "10" H 5770 2355 50  0000 L CNN
-F 2 "" V 5630 2400 50  0001 C CNN
+F 2 "Resistor_THT:R_Axial_DIN0207_L6.3mm_D2.5mm_P10.16mm_Horizontal" V 5630 2400 50  0001 C CNN
 F 3 "~" H 5700 2400 50  0001 C CNN
 	1    5700 2400
@@
 P 4650 1400
 F 0 "C12" H 4765 1446 50  0000 L CNN
-F 1 "4.7nF" H 4765 1355 50  0000 L CNN
-F 2 "" H 4688 1250 50  0001 C CNN
+F 1 "4700pF" H 4765 1355 50  0000 L CNN
+F 2 "Capacitor_THT:C_Disc_D5.1mm_W3.2mm_P5.00mm" H 4688 1250 50  0001 C CNN
 F 3 "~" H 4650 1400 50  0001 C CNN
 	1    4650 1400
@@
 F 0 "U3" H 5200 2350 50  0000 L CNN
 F 1 "LM386" H 5300 2000 50  0000 L CNN
-F 2 "" H 5250 2300 50  0001 C CNN
+F 2 "Package_DIP:DIP-8_W7.62mm_Socket" H 5250 2300 50  0001 C CNN
 F 3 "http://www.ti.com/lit/ds/symlink/lm386.pdf" H 5350 2400 50  0001 C CNN
 	1    5150 2200
@@
 F 0 "R11" V 4443 2100 50  0000 C CNN
 F 1 "10k" V 4534 2100 50  0000 C CNN
-F 2 "" V 4580 2100 50  0001 C CNN
+F 2 "Resistor_THT:R_Axial_DIN0207_L6.3mm_D2.5mm_P10.16mm_Horizontal" V 4580 2100 50  0001 C CNN
 F 3 "~" H 4650 2100 50  0001 C CNN
 	1    4650 2100
@@
 P 3750 2000
 F 0 "C10" H 3865 2046 50  0000 L CNN
-F 1 "1nF" H 3865 1955 50  0000 L CNN
-F 2 "" H 3788 1850 50  0001 C CNN
+F 1 "1000pF" H 3450 2100 50  0000 L CNN
+F 2 "Capacitor_THT:C_Disc_D5.0mm_W2.5mm_P5.00mm" H 3788 1850 50  0001 C CNN
 F 3 "~" H 3750 2000 50  0001 C CNN
 	1    3750 2000
@@
 F 0 "RV1" H 4281 2146 50  0000 R CNN
 F 1 "10k_pot" H 4281 2055 50  0000 R CNN
-F 2 "" H 4350 2100 50  0001 C CNN
+F 2 "Potentiometer_THT:Potentiometer_Bourns_PTV09A-2_Single_Horizontal" H 4350 2100 50  0001 C CNN
 F 3 "~" H 4350 2100 50  0001 C CNN
 	1    4350 2100
@@
 P 3950 1800
 F 0 "C11" V 3698 1800 50  0000 C CNN
-F 1 "100nF" V 3789 1800 50  0000 C CNN
-F 2 "" H 3988 1650 50  0001 C CNN
+F 1 "0.1uF" V 3789 1800 50  0000 C CNN
+F 2 "Capacitor_THT:C_Disc_D5.1mm_W3.2mm_P5.00mm" H 3988 1650 50  0001 C CNN
 F 3 "~" H 3950 1800 50  0001 C CNN
 	1    3950 1800
@@
 F 0 "R8" H 2470 1246 50  0000 L CNN
 F 1 "100" H 2470 1155 50  0000 L CNN
-F 2 "" V 2330 1200 50  0001 C CNN
+F 2 "Resistor_THT:R_Axial_DIN0207_L6.3mm_D2.5mm_P10.16mm_Horizontal" V 2330 1200 50  0001 C CNN
 F 3 "~" H 2400 1200 50  0001 C CNN
 	1    2400 1200
@@
 F 0 "J5" V 2718 2430 50  0000 L CNN
 F 1 "Conn_01x01" V 2763 2430 50  0001 L CNN
-F 2 "" H 2800 2350 50  0001 C CNN
+F 2 "Connector_PinHeader_2.54mm:PinHeader_1x01_P2.54mm_Vertical" H 2800 2350 50  0001 C CNN
 F 3 "~" H 2800 2350 50  0001 C CNN
 	1    2800 2350
@@
 F 0 "J4" H 2680 1696 50  0000 L CNN
 F 1 "Conn_01x01" V 2563 1780 50  0001 L CNN
-F 2 "" H 2600 1700 50  0001 C CNN
+F 2 "Connector_PinHeader_2.54mm:PinHeader_1x01_P2.54mm_Vertical" H 2600 1700 50  0001 C CNN
 F 3 "~" H 2600 1700 50  0001 C CNN
 	1    2600 1700
@@
 F 0 "J3" V 1918 2480 50  0000 L CNN
 F 1 "Conn_01x01" V 1963 2480 50  0001 L CNN
-F 2 "" H 2000 2400 50  0001 C CNN
+F 2 "Connector_PinHeader_2.54mm:PinHeader_1x01_P2.54mm_Vertical" H 2000 2400 50  0001 C CNN
 F 3 "~" H 2000 2400 50  0001 C CNN
 	1    2000 2400
@@
 F 0 "R9" H 2470 1546 50  0000 L CNN
 F 1 "100k" H 2470 1455 50  0000 L CNN
-F 2 "" V 2330 1500 50  0001 C CNN
+F 2 "Resistor_THT:R_Axial_DIN0207_L6.3mm_D2.5mm_P10.16mm_Horizontal" V 2330 1500 50  0001 C CNN
 F 3 "~" H 2400 1500 50  0001 C CNN
 	1    2400 1500
@@
 F 0 "R10" H 2470 1996 50  0000 L CNN
 F 1 "10M" H 2470 1905 50  0000 L CNN
-F 2 "" V 2330 1950 50  0001 C CNN
+F 2 "Resistor_THT:R_Axial_DIN0207_L6.3mm_D2.5mm_P10.16mm_Horizontal" V 2330 1950 50  0001 C CNN
 F 3 "~" H 2400 1950 50  0001 C CNN
 	1    2400 1950
@@
 P 2200 2150
 F 0 "C8" V 1948 2150 50  0000 C CNN
-F 1 "1nF" V 2039 2150 50  0000 C CNN
-F 2 "" H 2238 2000 50  0001 C CNN
+F 1 "1000pF" V 2039 2150 50  0000 C CNN
+F 2 "Capacitor_THT:C_Disc_D5.0mm_W2.5mm_P5.00mm" H 2238 2000 50  0001 C CNN
 F 3 "~" H 2200 2150 50  0001 C CNN
 	1    2200 2150
@@
 F 0 "R7" H 1720 1996 50  0000 L CNN
 F 1 "10M" H 1720 1905 50  0000 L CNN
-F 2 "" V 1580 1950 50  0001 C CNN
+F 2 "Resistor_THT:R_Axial_DIN0207_L6.3mm_D2.5mm_P10.16mm_Horizontal" V 1580 1950 50  0001 C CNN
 F 3 "~" H 1650 1950 50  0001 C CNN
 	1    1650 1950
@@
 F 0 "C7" H 965 2046 50  0000 L CNN
 F 1 "100pF" H 965 1955 50  0000 L CNN
-F 2 "" H 888 1850 50  0001 C CNN
+F 2 "Capacitor_THT:C_Disc_D5.0mm_W2.5mm_P5.00mm" H 888 1850 50  0001 C CNN
 F 3 "~" H 850 2000 50  0001 C CNN
 	1    850  2000
@@
 F 0 "D3" H 1400 2366 50  0000 C CNN
 F 1 "BAT41" H 1400 2275 50  0000 C CNN
-F 2 "" H 1400 2150 50  0001 C CNN
+F 2 "Diode_THT:D_DO-35_SOD27_P7.62mm_Horizontal" H 1400 2150 50  0001 C CNN
 F 3 "~" H 1400 2150 50  0001 C CNN
 	1    1400 2150
@@
 F 0 "R6" H 920 2346 50  0000 L CNN
 F 1 "10k" H 920 2255 50  0000 L CNN
-F 2 "" V 780 2300 50  0001 C CNN
+F 2 "Resistor_THT:R_Axial_DIN0207_L6.3mm_D2.5mm_P10.16mm_Horizontal" V 780 2300 50  0001 C CNN
 F 3 "~" H 850 2300 50  0001 C CNN
 	1    850  2300
-	1    0    0    -1
-$EndComp
-$Comp
-L Device:Antenna AE1
-U 1 1 5E7AB9F8
-P 850 1650
-F 0 "AE1" H 930 1639 50  0000 L CNN
-F 1 "Antenna" H 930 1548 50  0000 L CNN
-F 2 "" H 850 1650 50  0001 C CNN
-F 3 "~" H 850 1650 50  0001 C CNN
-	1    850  1650
 	1    0    0    -1
 $EndComp
@@
 F 0 "C16" H 5518 1696 50  0000 L CNN
 F 1 "1uF" H 5518 1605 50  0000 L CNN
-F 2 "" H 5438 1500 50  0001 C CNN
+F 2 "Capacitor_THT:CP_Radial_D5.0mm_P2.00mm" H 5438 1500 50  0001 C CNN
 F 3 "~" H 5400 1650 50  0001 C CNN
 	1    5400 1650
@@
 Wire Wire Line
 	5150 1500 5400 1500
+$Comp
+L Connector:Conn_Coaxial J6
+U 1 1 5E8326D9
+P 850 1650
+F 0 "J6" V 1087 1579 50  0000 C CNN
+F 1 "Conn_Coaxial" V 996 1579 50  0000 C CNN
+F 2 "homebrew:MOLEX_0731713150" H 850 1650 50  0001 C CNN
+F 3 " ~" H 850 1650 50  0001 C CNN
+	1    850  1650
+	0    -1   -1   0
+$EndComp
+$Comp
+L power:GND #PWR0102
+U 1 1 5E833EDC
+P 1050 1650
+F 0 "#PWR0102" H 1050 1400 50  0001 C CNN
+F 1 "GND" H 1055 1477 50  0000 C CNN
+F 2 "" H 1050 1650 50  0001 C CNN
+F 3 "" H 1050 1650 50  0001 C CNN
+	1    1050 1650
+	1    0    0    -1
+$EndComp
 $EndSCHEMATC

Commit message: First pass at layout
Parts:
- R12: value 1.2k -> 1.3k
- U3: footprint Package_DIP:DIP-8_W7.62mm_Socket -> Package_DIP:DIP-8_W7.62mm
Changed lines of the file:
@@
 P 5100 3150
 F 0 "R12" V 4893 3150 50  0000 C CNN
-F 1 "1.2k" V 4984 3150 50  0000 C CNN
+F 1 "1.3k" V 4984 3150 50  0000 C CNN
 F 2 "Resistor_THT:R_Axial_DIN0207_L6.3mm_D2.5mm_P10.16mm_Horizontal" V 5030 3150 50  0001 C CNN
 F 3 "~" H 5100 3150 50  0001 C CNN
@@
 F 0 "U3" H 5200 2350 50  0000 L CNN
 F 1 "LM386" H 5300 2000 50  0000 L CNN
-F 2 "Package_DIP:DIP-8_W7.62mm_Socket" H 5250 2300 50  0001 C CNN
+F 2 "Package_DIP:DIP-8_W7.62mm" H 5250 2300 50  0001 C CNN
 F 3 "http://www.ti.com/lit/ds/symlink/lm386.pdf" H 5350 2400 50  0001 C CNN
 	1    5150 2200
