File: all-through-hole/all-through-hole.kicad_pcb (KiCad board)
At the start: 2 copper layers, 96.5 x 79 mm, 53 parts, among them J1 Conn_01x01, J2 Conn_01x01, J3 Conn_01x01, J4 Conn_01x01, J5 Conn_01x01, J6 Conn_Coaxial, Q1 2N4401, SW1 SW_SPST, SW2 SW_SPST, U1 MC34063AP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

Commit message: Hardware v1.0
Routing:
- added copper zone on F.Cu, net +9V
- added copper zone on F.Cu, net Net-(A1-Pad1)
Other:
- board text added: "+"
- board text added: "-"
- board text added: "10V"
- board text added: "9V"
- board text added: "GAIN"
- board text added: "PWR"
- board text added: "TP1"
- board text added: "TP2"
- board text added: "TP3"
- board text added: "VOLUME"
- board text added: "all band receiver v1.0"
